File: AD3 Front End Amplifier.kicad_sch (KiCad schematic)
At the start: 48 parts, among them IC101 XC6901D501MR-G, J101 CH1, J102 CH2, J103 W1, J104 W2, J105 Conn_01x15_Pin, J106 Conn_01x15_Socket, J107 Conn_01x15_Pin, J108 Conn_01x15_Socket, SW101 AC/DC, SW102 AC/DC, SW103 50, SW104 50, U101 MIC5504-2.5YM5, U102 OPA356xxDBV, U103 OPA356xxDBV, U104 OPA356xxDBV, U105 OPA356xxDBV

Commit message: v2 gerbers and pdf schematics
Parts:
- removed C105, C106: 10n, Capacitor_THT:C_Rect_L7.0mm_W2.5mm_P5.00mm, symbol Device:C_Small
- removed C109, C110, C111, C112, C113, C114, C115, C116: 10u, Capacitor_SMD:C_0603_1608Metric_Pad1.08x0.95mm_HandSolder, symbol Device:C_Small
- removed J101: CH1, Connector_Coaxial:BNC_Amphenol_B6252HB-NPP3G-50_Horizontal, symbol Connector:Conn_Coaxial
- removed J102: CH2, Connector_Coaxial:BNC_Amphenol_B6252HB-NPP3G-50_Horizontal, symbol Connector:Conn_Coaxial
- removed R102, R103: 1M, Resistor_SMD:R_0805_2012Metric_Pad1.20x1.40mm_HandSolder, symbol Device:R_Small_US
- removed R104, R105: 100, Resistor_SMD:R_0402_1005Metric_Pad0.72x0.64mm_HandSolder, symbol Device:R_Small_US
- removed R106, R107, R109, R111, R112, R113: 402, Resistor_SMD:R_0402_1005Metric_Pad0.72x0.64mm_HandSolder, symbol Device:R_Small_US
- removed R108, R110, R114, R115: 22, Resistor_SMD:R_0402_1005Metric_Pad0.72x0.64mm_HandSolder, symbol Device:R_Small_US
- removed SW101, SW102: AC/DC, Button_Switch_THT:SW_DIP_SPSTx01_Slide_9.78x4.72mm_W7.62mm_P2.54mm, symbol Switch:SW_SPST
- removed SW103, SW104: 50, Button_Switch_THT:SW_DIP_SPSTx01_Slide_9.78x4.72mm_W7.62mm_P2.54mm, symbol Switch:SW_SPST
- removed U102, U103, U104, U105: OPA356xxDBV, Package_TO_SOT_SMD:SOT-23-5, symbol Amplifier_Operational:OPA356xxDBV
- added C121, C122, C123, C124: 1u, Capacitor_SMD:C_0402_1005Metric_Pad0.74x0.62mm_HandSolder, symbol Device:C_Small
- added FB101, FB102: FerriteBead_Small, Inductor_SMD:L_0603_1608Metric_Pad1.05x0.95mm_HandSolder, symbol Device:FerriteBead_Small
- C117: renamed from C101; value 10u -> 1u; footprint Capacitor_SMD:C_0603_1608Metric_Pad1.08x0.95mm_HandSolder -> Capacitor_SMD:C_0402_1005Metric_Pad0.74x0.62mm_HandSolder
- C118: renamed from C102; value 10u -> 1u; footprint Capacitor_SMD:C_0603_1608Metric_Pad1.08x0.95mm_HandSolder -> Capacitor_SMD:C_0402_1005Metric_Pad0.74x0.62mm_HandSolder
- C119: renamed from C107; footprint Capacitor_SMD:C_0603_1608Metric_Pad1.08x0.95mm_HandSolder -> Capacitor_SMD:C_0402_1005Metric_Pad0.74x0.62mm_HandSolder
- C120: renamed from C108; footprint Capacitor_SMD:C_0603_1608Metric_Pad1.08x0.95mm_HandSolder -> Capacitor_SMD:C_0402_1005Metric_Pad0.74x0.62mm_HandSolder
- renumbered IC101 to IC103, R116 to R117, R117 to R118, U101 to U105
Connections:
- net GND: now also C121.2, C122.2, C123.2, C124.2
- net V+: now also C124.1, FB102.2; no longer J107.4 (Pin_4), J108.4 (Pin_4)
- net V-: now also C122.1, FB101.2; no longer J105.4 (Pin_4), J106.4 (Pin_4)
- new net V+_CONN: C123.1, FB102.1, J107.4 (Pin_4), J108.4 (Pin_4)
- new net V-_CONN: C121.1, FB101.1, J105.4 (Pin_4), J106.4 (Pin_4)
Other:
- added sheet CH1 (CH1.kicad_sch)
- added sheet CH2 (CH1.kicad_sch)
- moved on the sheet: J103, J104, R117, R118

Commit message: v3 done
Parts:
- renumbered C121 to C101, C123 to C102, C122 to C103, C124 to C104, C117 to C105, C118 to C106, C119 to C107, C120 to C108, IC103 to IC101, J103 to J101, J104 to J102, J105 to J103, J106 to J104, J107 to J105, J108 to J106, R117 to R101, R118 to R102, U105 to U101
